File: RC1 Keypad MX/RC1 Keypad MX.sch (KiCad schematic (older format))
At the start: 26 parts, among them J1 KB, SW1 Ø, SW10 3, SW11 A, SW12 DA, SW13 4, SW14 B, SW15 +, SW16 5, SW17 C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

Commit message: MX Keypad now matches Commodore Kim-1
Parts:
- removed SW22: SST, Buttons_Switches_THT:SW_DIP_x1_W7.62mm_Slide, symbol SW_SPST
- added SW22: SST, Buttons_Switches_THT:SW_DIP_x1_W7.62mm_Slide, symbol SW_DIP_x01
- J1: symbol Conn_02x08_Counter_Clockwise -> RC1_Keypad_Port
Connections:
- net LED: no longer names the net of D1.1 (K), J1.14 (Pin_14)
- net RS: no longer names the net of J1.13 (Pin_13), SW23.2
- net SST_IN: no longer names the net of J1.16 (Pin_16)
- net SST_IN: now also SW22.1
- net SST_OUT: no longer names the net of J1.15 (Pin_15)
- net SST_OUT: now also SW22.2
- net ST: no longer names the net of J1.12 (Pin_12), SW24.2
- net VCC: no longer names the net of D1.2 (A), J1.11 (Pin_11), SW23.1, SW24.1
Other:
- note added: "The keypad module for the RC One computer, has the classic KIM-1 layout with a\ncustom connector. This is the MX version featuring Cherry MX key switches, larger and\nmore comfortable than the standard keys at an increased cost. See the non-MX version\nfor a cheaper alternative."
- note removed: "The keypad module for the RC One computer, has the classic KIM-1 layout with a\ncustom connector. This is the MX version featuring Cherry MX key switches, larger and\nmore comfortable than the standard keys at the cost of increased PCB costs."
- moved on the sheet: D1, SW1, SW10, SW11, SW12, SW13, SW14, SW15, SW16, SW17, SW18, SW19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
