File: RC1 CPU/RC1 CPU.kicad_pcb (KiCad board)
At the start: 2 copper layers, 99.1 x 99.1 mm, 47 parts, among them J1 Expansion, J2 RC1_UI_Port, J3 BARREL_JACK, M1 Mounting, M2 Mounting, M3 Mounting, M4 Mounting, U1 WD65C02, U2 HM62256BLP-7, U3 28C256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

Commit message: Eliminated 74LS145 from CPU module
Parts:
- removed R4, R5, R8: 1k, Resistors_THT:R_Axial_DIN0207_L6.3mm_D2.5mm_P10.16mm_Horizontal
- added J4: K1-4, Pin_Headers:Pin_Header_Straight_1x04_Pitch2.54mm, F.Cu at (141.0, 61.6)
- U1: value WD65C02 -> 6502
- U7: value 74LS145 -> 74LS138
- moved JP7 1.27 mm to (179.1, 120.7)
- moved JP8 0.63 mm to (191.1, 120.7)
Connections:
- net Net-(U9-Pad6) renamed /W/~R
- J1 pad 38: IO3 -> ~IO3
- J1 pad 39: TAPE -> (no net)
- J2 pad 20: TAPE -> (no net)
- U1 pad 38: (no net) -> VCC
- U4 pad 36: RAM_SEL -> ~RAM_SEL
- U5 pad 10: RAM_SEL -> ~RAM_SEL
- U5 pad 4: Net-(U5-Pad4) -> Net-(U5-Pad11)
- U5 pad 5: Net-(U5-Pad4) -> Net-(U5-Pad11)
- U5 pad 6: IO3 -> ~RAM_SEL
- U7 pad 1: Net-(JP3-Pad1) -> /A10
- U7 pad 10: (no net) -> K5
- U7 pad 11: (no net) -> Net-(J4-Pad4)
- U7 pad 12: /DEN -> Net-(J4-Pad3)
- U7 pad 13: /A12 -> Net-(J4-Pad2)
- U7 pad 14: /A11 -> Net-(J4-Pad1)
- U7 pad 15: /A10 -> Net-(JP3-Pad1)
- U7 pad 2: Net-(JP3-Pad1) -> /A11
- U7 pad 3: Net-(JP3-Pad1) -> /A12
- U7 pad 4: Net-(JP3-Pad1) -> /DEN
- U7 pad 5: Net-(JP3-Pad1) -> /DEN
- U7 pad 6: K5 -> VCC
- U7 pad 7: Net-(JP4-Pad1) -> Net-(U7-Pad7)
- U7 pad 9: Net-(JP4-Pad1) -> Net-(U7-Pad9)
- U8 pad 11: Net-(U5-Pad4) -> ~IO3
- U9 pad 1: Net-(U5-Pad11) -> Net-(U7-Pad9)
- U9 pad 11: (no net) -> Net-(JP4-Pad1)
- U9 pad 12: GND -> Net-(U9-Pad12)
- U9 pad 13: GND -> Net-(U9-Pad12)
- U9 pad 2: Net-(U5-Pad11) -> Net-(U7-Pad7)
- U9 pad 3: RAM_SEL -> Net-(U9-Pad12)
Routing:
- net IO3: track 192.8 -> 0.00 mm, vias 10 -> 0
- net ~IO3: track 0.00 -> 187.3 mm, vias 0 -> 5
- net RAM_SEL: track 102.2 -> 0.00 mm, vias 6 -> 0
- net ~RAM_SEL: track 0.00 -> 101.1 mm, vias 0 -> 7
- net K5: track 101.4 -> 15.1 mm, vias 5 -> 0
- net Net-(U7-Pad7): track 0.00 -> 55.4 mm, vias 0 -> 2
- net VCC: track 494.5 -> 548.6 mm, vias 9 -> 8
- net Net-(U7-Pad9): track 0.00 -> 50.7 mm, vias 0 -> 2
- net TAPE: track 39.2 -> 0.00 mm, vias 2 -> 0
- net Net-(U5-Pad4): track 14.5 -> 0.00 mm
- net Net-(J4-Pad2): track 0.00 -> 13.1 mm
- net Net-(J4-Pad4): track 0.00 -> 13.1 mm
- net Net-(J4-Pad1): track 0.00 -> 13.1 mm
- net Net-(J4-Pad3): track 0.00 -> 12.5 mm
- net Net-(JP4-Pad1): track 100.9 -> 90.3 mm
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Other:
- board text added: "$0000 - $03FF"
- board text added: "$0000 - $1FFF OPTIONAL $2000 - $3FFF $4000 - $5FFF $6000 - $7FFF"
- board text added: "$1740 $1741 $1742 $1743"
- board text added: "$1740 - $17FF"
- board text added: "$1744 $1745 $1746 $1747"
- board text added: "$174C $174D $174E $174F"
- board text added: "$1780 - $17FF"
- board text added: "$1800 - $FFFF"
- board text added: "$E000 - $FFFF"
- board text added: "$FFFA $17FA $FFFC $FFFE $17FE"
- board text added: "$FFFB $17FB $FFFD $FFFF $17FF"
- board text added: "/1 /8 /64 /1024"
- board text added: "/1 int. /8 int. /64 int. /1024 int."
- board text added: "1-2 Standalone 2-3 65K Expansion"
- board text added: "6502 CPU"
- board text added: "6532 RIOT"
- board text added: "65K EXPANSION"
- board text added: "8K0"
- board text added: "A13"
- board text added: "A14"
- board text added: "ADDRESS DECODER"
- board text added: "CPU Revision B"
- board text added: "EEPROM"
- board text added: "INTERRUPT"
- board text added: "K5"
- board text added: "MEMORY DECODING"
- board text added: "NAND GATES"
- board text added: "NMI RST IRQ"
- board text added: "OSCILLATOR"
- board text added: "Port A Port A DDR Port B Port B DDR"
- board text added: "REGISTERS"
- board text added: "STATIC RAM"
- board text added: "SWITCH DEBOUNCE"
- board text added: "TIMER"
- board text added: "VECTORS"
- board text removed: "CPU Revision A"
