File: RC1 CPU/RC1 CPU.sch (KiCad schematic (older format))
At the start: 45 parts, among them J1 Expansion, J2 RC1_UI_Port, J3 BARREL_JACK, J4 K1-4, M1 Mounting, M2 Mounting, M3 Mounting, M4 Mounting, U1 6502, U2 HM62256BLP-7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

Commit message: CPU/UI updated to KiCad 5
Parts:
- C1, C10, C11, C2, C3, C4, C5, C6, C7, C8, C9: symbol C -> Device:C
- J1: symbol RC1_Backplane -> rc1_backplane:RC1_Backplane
- J2: symbol RC1_UI_Port -> rc1_ui_port:RC1_UI_Port
- J3: symbol BARREL_JACK -> RC1-CPU-rescue:BARREL_JACK
- J4: symbol Conn_01x04 -> conn:Conn_01x04
- JP1, JP2: symbol Jumper_NO_Small -> Device:Jumper_NO_Small
- JP3, JP4, JP7, JP8: symbol Jumper_NC_Dual -> Device:Jumper_NC_Dual
- M1, M2, M3, M4: symbol Mounting -> mounting:Mounting
- R1, R10, R11, R12, R2, R3, R6, R7, R9: symbol R -> Device:R
- RN1: symbol R_Network08 -> Device:R_Network08
- U1: symbol 6502 -> 6502:6502
- U2: symbol HM62256BLP-7 -> memory:HM62256BLP-7
- U3: symbol 28C256 -> 28c256:28C256
- U4: symbol R6532 -> 65xx:R6532
- U5, U9: symbol 74LS00 -> RC1-CPU-rescue:74LS00
- U6: symbol LM556 -> linear:LM556
- U7, U8: symbol 74LS138 -> RC1-CPU-rescue:74LS138
- X1: symbol ACO-xxxMHz -> Oscillators:ACO-xxxMHz
Connections:
- wire segments 364 -> 404
