File: RC1 Project Examples/LED Cube/LED Cube.kicad_pcb (KiCad board)
At the start: 2 copper layers, 99.1 x 69.2 mm, 43 parts, among them J1 Signals, J5 Port A, J6 Port B, M1 Mounting, M2 Mounting, M3 Mounting, Q1 PN2222A, Q2 PN2222A, Q3 PN2222A, Q4 PN2222A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

Commit message: LED Cube 4x4 finishing touches
Parts:
- moved R13 10.5 mm to (137.2, 132.1), turned to 90 degrees
- moved R14 5.24 mm to (134.0, 132.1), turned to 90 degrees
Routing:
- net VCC: track 126.9 -> 175.8 mm
- net /PB7: track 100.0 -> 97.9 mm, vias 2 -> 0
- net /PB6: track 79.1 -> 80.9 mm, vias 2 -> 0
- net /PB4: track 71.8 -> 71.1 mm
- net /PB5: track 67.0 -> 66.3 mm
- net /PB3: track 77.4 -> 76.7 mm
- net /PB2: track 82.5 -> 81.7 mm
Other:
- board text added: "4x 2N2222"
- board text added: "A(+)"
- board text added: "Assemble lattice on this side, wrap anode (+) around metal rod. Solder cathodes together."
- board text added: "C(-)"
- board text added: "Create 4 layers separately, mount each on rods and solder at suitable heights."
- board text added: "D0"
- board text added: "D7"
- board text added: "DATA LATCH ANODES 1-8"
- board text added: "DATA LATCH ANODES 9-16"
- board text added: "L0"
- board text added: "L1"
- board text added: "L2"
- board text added: "L3"
- board text added: "LED Cube 4x4"
- board text added: "SW"
- board text added: "U1 ~CP"
- board text added: "U2 ~CP"
- board text removed: "LED Cube"
- board text removed: "PA0"
- board text removed: "PA1"
- board text removed: "PA2"
- board text removed: "PA3"
- board text removed: "PA4"
- board text removed: "PA5"
- board text removed: "PA6"
- board text removed: "PA7"
- board text removed: "PB0"
- board text removed: "PB1"
- board text removed: "PB2"
- board text removed: "PB3"
- board text removed: "PB4"
- board text removed: "PB5"
- board text removed: "PB6"
- board text removed: "PB7"
