File: RC1 65K Expansion/RC1 65K Expansion.kicad_pcb (KiCad board)
At the start: 2 copper layers, 99.1 x 55.2 mm, 23 parts, among them J1 Expansion, J2 External IO, J3 Extra, J4 K1-K4, J5 LOW RAM, U1 74LS138, U2 74LS138, U3 74LS08, U4 R6532, U5 74LS08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

Commit message: 65K Expansion silkscreen updated
Other:
- board text added: "6532 RIOT KIM-1 Application I/O"
- board text added: "8K0-8K7 ADDRESS DECODER"
- board text added: "K0-K7 ADDRESS DECODER"
- board text added: "NAND GATES"
- board text added: "RAM SELECT LOGIC"
Changed lines of the file:
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@@
     (area 91.364999 84.379999 190.575001 139.775001)
     (thickness 1.6)
-    (drawings 176)
+    (drawings 226)
     (tracks 886)
     (zones 0)
@@
     )
   )
+  (gr_line (start 186.69 132.08) (end 186.69 123.19) (angle 90) (layer B.SilkS) (width 0.2))
+  (gr_line (start 190.5 132.08) (end 186.69 132.08) (angle 90) (layer B.SilkS) (width 0.2))
+  (gr_line (start 190.5 123.19) (end 190.5 132.08) (angle 90) (layer B.SilkS) (width 0.2))
+  (gr_line (start 186.69 123.19) (end 190.5 123.19) (angle 90) (layer B.SilkS) (width 0.2))
+  (gr_line (start 175.26 132.08) (end 171.45 132.08) (angle 90) (layer B.SilkS) (width 0.2))
+  (gr_line (start 175.26 120.65) (end 175.26 132.08) (angle 90) (layer B.SilkS) (width 0.2))
+  (gr_line (start 171.45 120.65) (end 175.26 120.65) (angle 90) (layer B.SilkS) (width 0.2))
+  (gr_line (start 171.45 132.08) (end 171.45 120.65) (angle 90) (layer B.SilkS) (width 0.2))
+  (gr_text "6532 RIOT\n\nKIM-1 Application I/O" (at 119.38 120.015) (layer B.SilkS)
+    (effects (font (size 0.8 0.8) (thickness 0.1)) (justify mirror))
+  )
+  (gr_line (start 144.145 112.395) (end 142.875 112.395) (angle 90) (layer B.SilkS) (width 0.2))
+  (gr_line (start 144.145 127.635) (end 144.145 112.395) (angle 90) (layer B.SilkS) (width 0.2))
+  (gr_line (start 142.875 127.635) (end 144.145 127.635) (angle 90) (layer B.SilkS) (width 0.2))
+  (gr_line (start 92.075 127.635) (end 93.345 127.635) (angle 90) (layer B.SilkS) (width 0.2))
+  (gr_line (start 92.075 112.395) (end 92.075 127.635) (angle 90) (layer B.SilkS) (width 0.2))
+  (gr_line (start 93.345 112.395) (end 92.075 112.395) (angle 90) (layer B.SilkS) (width 0.2))
+  (gr_line (start 184.785 85.725) (end 184.785 86.995) (angle 90) (layer B.SilkS) (width 0.2))
+  (gr_line (start 177.165 85.725) (end 184.785 85.725) (angle 90) (layer B.SilkS) (width 0.2))
+  (gr_line (start 177.165 86.995) (end 177.165 85.725) (angle 90) (layer B.SilkS) (width 0.2))
+  (gr_line (start 169.545 85.725) (end 169.545 86.995) (angle 90) (layer B.SilkS) (width 0.2))
+  (gr_line (start 161.925 85.725) (end 169.545 85.725) (angle 90) (layer B.SilkS) (width 0.2))
+  (gr_line (start 161.925 86.995) (end 161.925 85.725) (angle 90) (layer B.SilkS) (width 0.2))
+  (gr_line (start 184.785 104.775) (end 184.785 103.505) (angle 90) (layer B.SilkS) (width 0.2))
+  (gr_line (start 177.165 104.775) (end 184.785 104.775) (angle 90) (layer B.SilkS) (width 0.2))
+  (gr_line (start 177.165 103.505) (end 177.165 104.775) (angle 90) (layer B.SilkS) (width 0.2))
+  (gr_line (start 169.545 104.775) (end 169.545 103.505) (angle 90) (layer B.SilkS) (width 0.2))
+  (gr_line (start 161.925 104.775) (end 169.545 104.775) (angle 90) (layer B.SilkS) (width 0.2))
+  (gr_line (start 161.925 103.505) (end 161.925 104.775) (angle 90) (layer B.SilkS) (width 0.2))
+  (gr_line (start 184.785 132.08) (end 184.785 130.81) (angle 90) (layer B.SilkS) (width 0.2))
+  (gr_line (start 177.165 132.08) (end 184.785 132.08) (angle 90) (layer B.SilkS) (width 0.2))
+  (gr_line (start 177.165 130.81) (end 177.165 132.08) (angle 90) (layer B.SilkS) (width 0.2))
+  (gr_line (start 169.545 132.08) (end 169.545 130.81) (angle 90) (layer B.SilkS) (width 0.2))
+  (gr_line (start 161.925 132.08) (end 169.545 132.08) (angle 90) (layer B.SilkS) (width 0.2))
+  (gr_line (start 161.925 130.81) (end 161.925 132.08) (angle 90) (layer B.SilkS) (width 0.2))
+  (gr_line (start 154.305 129.54) (end 154.305 128.27) (angle 90) (layer B.SilkS) (width 0.2))
+  (gr_line (start 146.685 129.54) (end 154.305 129.54) (angle 90) (layer B.SilkS) (width 0.2))
+  (gr_line (start 146.685 128.27) (end 146.685 129.54) (angle 90) (layer B.SilkS) (width 0.2))
+  (gr_line (start 184.785 110.49) (end 184.785 111.76) (angle 90) (layer B.SilkS) (width 0.2))
+  (gr_line (start 177.165 110.49) (end 184.785 110.49) (angle 90) (layer B.SilkS) (width 0.2))
+  (gr_line (start 177.165 111.76) (end 177.165 110.49) (angle 90) (layer B.SilkS) (width 0.2))
+  (gr_line (start 169.545 110.49) (end 169.545 111.76) (angle 90) (layer B.SilkS) (width 0.2))
+  (gr_line (start 161.925 110.49) (end 169.545 110.49) (angle 90) (layer B.SilkS) (width 0.2))
+  (gr_line (start 161.925 111.76) (end 161.925 110.49) (angle 90) (layer B.SilkS) (width 0.2))
+  (gr_line (start 154.305 110.49) (end 154.305 111.76) (angle 90) (layer B.SilkS) (width 0.2))
+  (gr_line (start 146.685 110.49) (end 154.305 110.49) (angle 90) (layer B.SilkS) (width 0.2))
+  (gr_line (start 146.685 111.76) (end 146.685 110.49) (angle 90) (layer B.SilkS) (width 0.2))
+  (gr_text "RAM\nSELECT\nLOGIC" (at 150.495 120.015) (layer B.SilkS)
+    (effects (font (size 0.8 0.8) (thickness 0.1)) (justify mirror))
+  )
+  (gr_text "RAM\nSELECT\nLOGIC" (at 165.735 95.25) (layer B.SilkS)
+    (effects (font (size 0.8 0.8) (thickness 0.1)) (justify mirror))
+  )
+  (gr_text "NAND\nGATES" (at 180.975 95.25) (layer B.SilkS)
+    (effects (font (size 0.8 0.8) (thickness 0.1)) (justify mirror))
+  )
+  (gr_text "K0-K7\n\nADDRESS\nDECODER" (at 165.735 121.285) (layer B.SilkS)
+    (effects (font (size 0.8 0.8) (thickness 0.1)) (justify mirror))
+  )
+  (gr_text "8K0-8K7\n\nADDRESS\nDECODER" (at 180.975 121.285) (layer B.SilkS)
+    (effects (font (size 0.8 0.8) (thickness 0.1)) (justify mirror))
+  )
   (gr_line (start 119.38 95.25) (end 111.76 95.25) (angle 90) (layer F.SilkS) (width 0.2))
