File: RC1 Real Time Clock/RC1 Real Time Clock.sch (KiCad schematic (older format))
At the start: 28 parts, among them J1 Expansion, J2 ADDRESS, J3 SQW, J4 Battery, SW1 RAM_CLR, U1 74LS04, U2 DS12885, U3 74LS14, U4 74LS27, U5 74LS138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

Commit message: Fixed RTC address calculations
Connections:
- net 8K1 renamed 4K3
- net 8K2 renamed 4K5
- net 8K3 renamed 4K7
- net 8K4 renamed 4K9
- net 8K5 renamed 4KB
- net 8K6 renamed 4KD
Other:
- note added: "$3000"
- note added: "$5000"
- note added: "$7000"
- note added: "$9000"
- note added: "$B000"
- note added: "$D000"
- note removed: "$2000"
- note removed: "$4000"
- note removed: "$6000"
- note removed: "$8000"
- note removed: "$A000"
- note removed: "$C000"
Changed lines of the file:
@@
 $EndComp
 Text Label 2550 2400 0    60   ~ 0
-8K1
+4K3
 Text Label 2550 2500 0    60   ~ 0
-8K2
+4K5
 Text Label 2550 2600 0    60   ~ 0
-8K3
+4K7
 Entry Wire Line
 	825  2200 925  2300
@@
 	825  2400 925  2500
 Text Notes 2800 2400 0    60   ~ 0
-$2000
+$3000
 Text Notes 2800 2500 0    60   ~ 0
-$4000
+$5000
 Text Notes 2800 2600 0    60   ~ 0
-$6000
+$7000
 Text Notes 2800 2700 0    60   ~ 0
-$8000
+$9000
 Text Notes 2800 2800 0    60   ~ 0
-$A000
+$B000
 Text Notes 2800 2900 0    60   ~ 0
-$C000
+$D000
 $Comp
 L C C4
@@
 	14250 7075 14350 7175
 Text Label 2550 2700 0    60   ~ 0
-8K4
+4K9
 Text Label 2550 2800 0    60   ~ 0
-8K5
+4KB
 Text Label 2550 2900 0    60   ~ 0
-8K6
+4KD
 NoConn ~ 14750 5675
 NoConn ~ 14750 5375
@@
 	10250 9175 10250 9050
 Wire Wire Line
-	9975 9050 10250 9050
+	10250 9050 9975 9050
 Wire Wire Line
 	9975 8475 9975 9125
