File: RC1 TMS9918A/RC1 TMS9918A.sch (KiCad schematic (older format))
At the start: 32 parts, among them J1 Expansion, J2 ADDRESS, J3 INT_SEL, J4 VIDEO, Q1 2N3904, U1 TMS9918A, U2 HM62256BLP-7, U3 74LS138, U4 74LS138, U5 74HCT04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

Commit message: TMS9918 layout
Parts:
- L1: footprint Inductors_THT:L_Axial_L6.6mm_D2.7mm_P10.16mm_Horizontal_Vishay_IM-2 -> Inductors_THT:L_Axial_L7.0mm_D3.3mm_P10.16mm_Horizontal_Fastron_MICC
Connections:
- net GND: now also C10.1, C9.1; no longer C10.2, C9.2
- net ~IRQ: now also J3.3 (Pin_3); no longer J3.1 (Pin_1)
- net ~NMI: now also J3.1 (Pin_1); no longer J3.3 (Pin_3)
- net at U1.40 (XTAL2), Y1.1: now also C10.2; no longer C10.1
- net at U1.39 (XTAL1), Y1.2: now also C9.2; no longer C9.1
- net VA0: now reaches U1.10 (AD0), U6.3 (D0), U7.3 (D0), U8.3 (D0)
- net VA7: now reaches U1.3 (AD7), U6.18 (D7), U7.18 (D7), U8.18 (D7)
- net VA6: now reaches U1.4 (AD6), U6.17 (D6), U7.17 (D6), U8.17 (D6)
- net VA5: now reaches U1.5 (AD5), U6.14 (D5), U7.14 (D5), U8.14 (D5)
- net VA4: now reaches U1.6 (AD4), U6.13 (D4), U7.13 (D4), U8.13 (D4)
- net VA3: now reaches U1.7 (AD3), U6.8 (D3), U7.8 (D3), U8.8 (D3)
- net VA2: now reaches U1.8 (AD2), U6.7 (D2), U7.7 (D2), U8.7 (D2)
- net VA1: now reaches U1.9 (AD1), U6.4 (D1), U7.4 (D1), U8.4 (D1)
- net ROW0: now reaches U2.10 (A0), U6.5 (O1)
- net COL5: now reaches U2.2 (A12), U7.16 (O6)
- net COL3: now reaches U2.21 (A10), U7.12 (O4)
- net COL4: now reaches U2.23 (A11), U7.15 (O5)
- net COL2: now reaches U2.24 (A9), U7.9 (O3)
- net COL1: now reaches U2.25 (A8), U7.6 (O2)
- net COL6: now reaches U2.26 (A13), U7.19 (O7)
- net COL0: now reaches U2.3 (A7), U7.5 (O1)
- net ROW6: now reaches U2.4 (A6), U6.19 (O7)
- net ROW5: now reaches U2.5 (A5), U6.16 (O6)
- net ROW4: now reaches U2.6 (A4), U6.15 (O5)
- net ROW3: now reaches U2.7 (A3), U6.12 (O4)
- net ROW2: now reaches U2.8 (A2), U6.9 (O3)
- net ROW1: now reaches U2.9 (A1), U6.6 (O2)
- net 4K3 renamed 4K2
- net 4K5 renamed 4K4
- net 4K7 renamed 4K6
- net 4K9 renamed 4K8
- net 4KB renamed 4KA
- net 4KD renamed 4KC
Other:
- note added: "Video Display Controller based on the TMS9918 chip from Texas Instruments, schematic\nbased on an earlier 6809-based build called Ultim809 with changes for 6502 CPU and\naddress decoding scheme for RC-ONE."
Changed lines of the file:
@@
 $EndComp
 Text Label 2725 2575 0    60   ~ 0
-4K3
+4K2
 Text Label 2725 2675 0    60   ~ 0
-4K5
+4K4
 Text Label 2725 2775 0    60   ~ 0
-4K7
+4K6
 Entry Wire Line
 	1000 2375 1100 2475
@@
 	14250 7075 14350 7175
 Text Label 2725 2875 0    60   ~ 0
-4K9
+4K8
 Text Label 2725 2975 0    60   ~ 0
-4KB
+4KA
 Text Label 2725 3075 0    60   ~ 0
-4KD
+4KC
 NoConn ~ 14750 5675
 NoConn ~ 14750 5375
@@
 Entry Wire Line
 	4225 5975 4125 6075
+Text Label 4100 6075 2    60   ~ 0
+~NMI
 Text Label 4100 5975 2    60   ~ 0
-~NMI
-Text Label 4100 6075 2    60   ~ 0
 ~IRQ
 $Comp
@@
 F 3 "" H 4375 6275 50  0001 C CNN
 	1    4375 6275
-	0    1    1    0
+	0    -1   -1   0
 $EndComp
 $Comp
@@
 F 3 "" H 4375 6675 50  0001 C CNN
 	1    4375 6675
-	0    1    1    0
+	0    -1   -1   0
 $EndComp
 $Comp
@@
 F 0 "L1" H 2300 8025 50  0000 L CNN
 F 1 "BEAD" H 2300 7925 50  0000 L CNN
-F 2 "Inductors_THT:L_Axial_L6.6mm_D2.7mm_P10.16mm_Horizontal_Vishay_IM-2" V 2155 7975 50  0001 C CNN
+F 2 "Inductors_THT:L_Axial_L7.0mm_D3.3mm_P10.16mm_Horizontal_Fastron_MICC" V 2155 7975 50  0001 C CNN
 F 3 "" H 2225 7975 50  0001 C CNN
 	1    2225 7975
@@
 	1    0    0    -1
 $EndComp
+Text Label 6600 4275 2    60   ~ 0
+VA0
+Text Label 6600 4375 2    60   ~ 0
+VA1
+Text Label 6600 4475 2    60   ~ 0
+VA2
+Text Label 6600 4575 2    60   ~ 0
+VA3
+Text Label 6600 4675 2    60   ~ 0
+VA4
+Text Label 6600 4775 2    60   ~ 0
+VA5
+Text Label 6600 4875 2    60   ~ 0
+VA6
+Text Label 6600 4975 2    60   ~ 0
+VA7
+Text Label 10050 4375 2    60   ~ 0
+ROW0
+Text Label 10050 4475 2    60   ~ 0
+ROW1
+Text Label 10050 4575 2    60   ~ 0
+ROW2
+Text Label 10050 4675 2    60   ~ 0
+ROW3
+Text Label 10050 4775 2    60   ~ 0
+ROW4
+Text Label 10050 4875 2    60   ~ 0
+ROW5
+Text Label 10050 4975 2    60   ~ 0
+ROW6
+Text Label 10050 5075 2    60   ~ 0
+COL0
+Text Label 10050 5175 2    60   ~ 0
+COL1
+Text Label 10050 5275 2    60   ~ 0
+COL2
+Text Label 10050 5375 2    60   ~ 0
+COL3
+Text Label 10050 5475 2    60   ~ 0
+COL4
+Text Label 10050 5575 2    60   ~ 0
+COL5
+Text Label 10050 5675 2    60   ~ 0
+COL6
+Text Notes 11825 10250 0    60   ~ 0
+Video Display Controller based on the TMS9918 chip from Texas Instruments, schematic\nbased on an earlier 6809-based build called Ultim809 with changes for 6502 CPU and\naddress decoding scheme for RC-ONE.
 $EndSCHEMATC
